File: vcdcl_main_board/vcdcl_main_board.sch (KiCad schematic (older format))
At the start: 57 parts, among them J1 Conn_01x03_Male, J10 Conn_01x01_Male, J11 Conn_01x01_Male, J2 Conn_01x01_Male, J3 Conn_01x01_Male, J4 Conn_01x01_Male, J5 Conn_01x01_Male, J6 Conn_01x01_Male, J7 Conn_01x01_Male, J8 Conn_01x01_Male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

Commit message: Both boards update
Parts:
- removed J1: Conn_01x03_Male, _сustom:LUT_FanPinHeader_1x03_P2.54mm_Vertical, symbol Connector:Conn_01x03_Male
- removed J10, J11, J2, J3, J4, J5, J6, J7, J8, J9: Conn_01x01_Male, _сustom:LUT_PinHeader_1x01_P2.54mm_Vertical, symbol Connector:Conn_01x01_Male
- added D1: D, symbol Device:D
- added F1, F2: 10, symbol Device:Fuse
- added J1, J10, J12, J13, J2, J3, J4, J5, J6, J7, J8, J9: Conn_01x01, _сustom:LUT_PinHeader_1x01_P2.54mm_Vertical, symbol Connector_Generic:Conn_01x01
- added J11: Conn_01x03, _сustom:LUT_FanPinHeader_1x03_P2.54mm_Vertical, symbol Connector_Generic:Conn_01x03
- added Q1, Q2, Q3, Q4: IRF3205, symbol Device:Q_NMOS_GDS
- added R27: 10k 1%, symbol Device:R
- added R28, R29, R30, R31: 51, symbol Device:R
- added R32, R33, R34, R35, R36, R37, R38, R39: 200m 1%, symbol Device:R
- R15, R17, R19, R21: value 20k 0.1% -> 16k 0.1%
- R16, R18, R20, R22: value 20k 0.1% -> 24k 0.1%
Connections:
- net GND: now also J11.1 (Pin_1), J8.1 (Pin_1), R36.2, R37.2, R38.2, R39.2
- net Gate0: now also J1.1 (Pin_1), R28.2
- net Gate1: now also J5.1 (Pin_1), R29.2
- net Gate2: now also J9.1 (Pin_1), R30.2
- net Gate3: now also J12.1 (Pin_1), R31.2
- net PortIn: now also J3.1 (Pin_1)
- net SR0: now also J2.1 (Pin_1), Q1.3 (S), R32.1
- net SR1: now also J6.1 (Pin_1), Q2.3 (S), R33.1
- net SR2: now also J10.1 (Pin_1), Q3.3 (S), R34.1
- net SR3: now also J13.1 (Pin_1), Q4.3 (S), R35.1
- net V+: now also J11.3 (Pin_3)
- net V-: now also J11.2 (Pin_2)
- net PortOut renamed PortOutC
- net PortOutC: now also J7.1 (Pin_1)
- new net: R32.2, R36.1
- new net: Q1.1 (G), R28.1
- new net: F2.2, Q1.2 (D), Q2.2 (D), Q3.2 (D), Q4.2 (D)
- new net: R33.2, R37.1
- new net: Q2.1 (G), R29.1
- new net: R34.2, R38.1
- new net: Q3.1 (G), R30.1
- new net: R35.2, R39.1
- new net: Q4.1 (G), R31.1
- new net: D1.2 (A), F1.2
- new net Load: D1.1 (K), F2.1, J4.1 (Pin_1), R27.2
- new net LoadRPP: F1.1
- new net PortOutV: R27.1
Other:
- note added: "Current reference\ngenerator"
- note added: "Input voltage divider"
- note added: "Interface"
- note added: "MOSFET\ndriver array"
- note added: "Output resistance: 10kΩ ±0.1%"
- note added: "Point-to-point construction"
- note removed: "Current reference generator."
- note removed: "Input voltage divider."
- note removed: "Interface."
- note removed: "MOSFET driver array."
- moved on the sheet: C5, C6, H1, H2, H3, H4, R15, R16, R17, R18, R19, R20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
