File: vcdcl_main_board/vcdcl_main_board.kicad_pcb (KiCad board)
At the start: 2 copper layers, 100 x 50 mm, 58 parts, among them J1 Conn_01x03_Male, J10 Conn_01x01_Male, J11 Conn_01x01_Male, J2 Conn_01x01_Male, J3 Conn_01x01_Male, J4 Conn_01x01_Male, J5 Conn_01x01_Male, J6 Conn_01x01_Male, J7 Conn_01x01_Male, J8 Conn_01x01_Male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

Commit message: Both boards update
Parts:
- removed J4, J8: Conn_01x01_Male, _сustom:LUT_PinHeader_1x01_P2.54mm_Vertical
- added J12: Conn_01x01, _сustom:LUT_PinHeader_1x01_P2.54mm_Vertical, F.Cu at (129.1, 96.9)
- added J13: Conn_01x01, _сustom:LUT_PinHeader_1x01_P2.54mm_Vertical, F.Cu at (134.1, 70.5)
- J1: value Conn_01x03_Male -> Conn_01x01; footprint _сustom:LUT_FanPinHeader_1x03_P2.54mm_Vertical -> _сustom:LUT_PinHeader_1x01_P2.54mm_Vertical
- J10, J2, J3, J5, J6, J7, J9: value Conn_01x01_Male -> Conn_01x01
- J11: value Conn_01x01_Male -> Conn_01x03; footprint _сustom:LUT_PinHeader_1x01_P2.54mm_Vertical -> _сustom:LUT_FanPinHeader_1x03_P2.54mm_Vertical
- R15, R17, R19, R21: value 20k 0.1% -> 16k 0.1%
- R16, R18, R20, R22: value 20k 0.1% -> 24k 0.1%
- moved J11 68.7 mm to (60.5, 93.3), turned to 90 degrees
- moved J7 44.5 mm to (130.1, 104.5)
- moved J3 39.7 mm to (85.9, 109.9)
- moved J6 35.6 mm to (98.6, 70.5)
- moved J5 34.9 mm to (93.5, 96.9)
- moved J2 27.2 mm to (80.8, 70.4)
- moved J10 27.1 mm to (116.4, 70.5)
- moved J9 17.9 mm to (111.4, 96.9)
- moved J1 15.7 mm to (75.7, 96.9), turned to 0 degrees
- moved G*** 0.36 mm to (66.6, 109.6)
Connections:
- J1 pad 1: GND -> Gate0
- J10 pad 1: Gate2 -> SR2
- J11 pad 1: Gate3 -> GND
- J2 pad 1: Gate0 -> SR0
- J3 pad 1: SR0 -> PortIn
- J5 pad 1: SR2 -> Gate1
- J6 pad 1: SR3 -> SR1
- J7 pad 1: PortIn -> PortOutC
- J9 pad 1: Gate1 -> Gate2
- R16 pad 1: PortOut -> PortOutC
- R18 pad 1: PortOut -> PortOutC
- R20 pad 1: PortOut -> PortOutC
- R22 pad 1: PortOut -> PortOutC
Routing:
- net PortOutC: track 0.00 -> 61.2 mm
- net PortOut: track 61.2 -> 0.00 mm
Other:
- board size 100 x 50 mm -> 100 x 115 mm
- board text added: "1.0 A/V"
- board text added: "100m"
- board text added: "10k"
- board text added: "OFF"
- board text added: "ON"
- board text added: "VCDCL Main PCB rev. 1.7"
- board text added: "Voltage-controlled DC load "Ozen""
- board text removed: "VCDCL Main PCB rev. 1.6"

Commit message: Append schematic pdf files
Other:
- board text added: "0.1"
- board text removed: "100m"
