File: vcdcl_supply_board/vcdcl_supply_board.sch (KiCad schematic (older format))
At the start: 19 parts, among them J1 Conn_01x02_Male, Q1 IRFR9024, Q2 Q_NPN_ECB, Q3 Q_NPN_BCE, SW1 SW_DIP_x01

Commit message: Supply board fixes
Parts:
- removed J1: Conn_01x02_Male, _сustom:LUT_PinHeader_1x02_P2.54mm_Vertical, symbol Connector:Conn_01x02_Male
- added C1: 1u, _сustom:LUT_C_Rect_L7.0mm_W4.5mm_P5.00mm, symbol Device:C
- added C2: 10u, _сustom:LUT_CP_Radial_D4.0mm_P2.00mm, symbol Device:CP
- added C3: 100u, _сustom:LUT_CP_Radial_D6.3mm_P2.50mm, symbol Device:CP
- added C6: 470u, _сustom:LUT_CP_Radial_D6.3mm_P2.50mm, symbol Device:CP
- added C7: 150u, _сustom:LUT_C_Rect_L10.3mm_W5.0mm_P7.50mm, symbol Device:C
- added H3, H4, H5, H6: MountingHole_Pad, MountingHole:MountingHole_3.2mm_M3_ISO7380_Pad, symbol Mechanical:MountingHole_Pad
- added J1, J2, J3, J4: Conn_01x01_Female, _сustom:LUT_PinHeader_1x01_P2.54mm_Vertical, symbol Connector:Conn_01x01_Female
- added J5: Conn_01x03, _сustom:LUT_FanPinHeader_1x03_P2.54mm_Vertical, symbol Connector_Generic:Conn_01x03
- added Q3: Q_NPN_ECB, _сustom:LUT_TO-92, symbol Device:Q_NPN_ECB
- added R1: 10, _сustom:LUT_R_L6.3mm_D2.5mm_P7.62mm_Horizontal, symbol Device:R
- added R10, R6: 5k 1%, _сustom:LUT_R_L6.3mm_D2.5mm_P7.62mm_Horizontal, symbol Device:R
- added R11: 5k, _сustom:LUT_R_L6.3mm_D2.5mm_P7.62mm_Horizontal, symbol Device:R
- added R3: 100k, _сustom:LUT_R_L6.3mm_D2.5mm_P7.62mm_Horizontal, symbol Device:R
- added R4: 1k, _сustom:LUT_R_L6.3mm_D2.5mm_P7.62mm_Horizontal, symbol Device:R
- added R7: 1k 1%, _сustom:LUT_R_L6.3mm_D2.5mm_P7.62mm_Horizontal, symbol Device:R
- added R8: 10k 1%, _сustom:LUT_R_L6.3mm_D2.5mm_P7.62mm_Horizontal, symbol Device:R
- added R9: 47, _сustom:LUT_R_L6.3mm_D2.5mm_P7.62mm_Horizontal, symbol Device:R
- added U1: TL431LP, _сustom:LUT_TO-92, symbol Reference_Voltage:TL431LP
- added U2: LM741, _сustom:LUT_DIP-8, symbol Amplifier_Operational:LM741
- C4: renamed from C1; value 100u -> 47u 63v; footprint _сustom:LUT_CP_Radial_D6.3mm_P2.50mm -> _сustom:LUT_CP_Radial_D8.0mm_P2.50mm
- C5: renamed from C3; value 470u -> 470u 16v
- D1: footprint _сustom:LUT_D_P7.62mm_Horizontal -> _сustom:LUT_D_P10.16mm_Horizontal
- R2: renamed from R1; value 1k -> 390
- R5: renamed from R2; value 10k -> 5k
- renumbered JFan1 to J6, Q3 to Q4
Connections:
- net +12V: now also J5.1 (Pin_1); no longer J6.1 (Pin_1)
- net Earth: now also C1.2, C2.2, C3.2, C6.2, C7.2, J1.1 (Pin_1), J2.1 (Pin_1), J5.2 (Pin_2), J5.3 (Pin_3), R10.2, R3.1, R7.2, U1.2 (A), U2.4 (V-); no longer J6.3 (Pin_3)
- net V+ renamed Vin
- net Vin: now also J3.1 (Pin_1), J4.1 (Pin_1), R1.2, R3.2
- new net: C1.1, C2.1, C3.1, Q3.2 (C), R1.1, R4.1
- new net: R6.2, R7.1, U1.1 (REF)
- new net: Q3.3 (B), R4.2, U1.3 (K)
- new net: R11.2, U2.2 (-)
- new net: R10.1, R8.2, U2.3 (+)
- new net: R11.1, R9.2, U2.6
- new net +15V: J6.3 (Pin_3), Q3.1 (E), R6.1, R8.1, U2.7 (V+)
- new net +5V: C6.1, C7.1, J6.1 (Pin_1), R9.1
Other:
- note added: "+5v reference generator."
- note added: "Input Protection Board"
- note added: "Interface"
- note added: "Mounting"
- note added: "Power Supply Board"
- moved on the sheet: C4, C5, D1, D2, D3, D4, F1, H1, H2, J6, JSup1, Q1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

Commit message: Both boards update
Parts:
- removed J1, J2, J3, J4: Conn_01x01_Female, _сustom:LUT_PinHeader_1x01_P2.54mm_Vertical, symbol Connector:Conn_01x01_Female
- added J1, J2, J3, J4: Conn_01x01, _сustom:LUT_PinHeader_1x01_P2.54mm_Vertical, symbol Connector_Generic:Conn_01x01
- C5: value 470u 16v -> 470u 25v
Connections:
- net Earth: now also J2.1 (Pin_1), J4.1 (Pin_1)
- net Vin renamed +19V
- net +19V: now also J1.1 (Pin_1), J3.1 (Pin_1)
Other:
- note added: "+5v reference generator"
- note removed: "+5v reference generator."
- moved on the sheet: H3, H5
Changed lines of the file:
@@
 Title ""
 Date ""
-Rev "1.3"
+Rev "1.4"
 Comp ""
 Comment1 ""
@@
 P 6650 2850
 F 0 "C5" H 6765 2896 50  0000 L CNN
-F 1 "470u 16v" H 6765 2805 50  0000 L CNN
+F 1 "470u 25v" H 6765 2805 50  0000 L CNN
 F 2 "_сustom:LUT_CP_Radial_D6.3mm_P2.50mm" H 6650 2850 50  0001 C CNN
 F 3 "~" H 6650 2850 50  0001 C CNN
 	1    6650 2850
 	1    0    0    -1
-$EndComp
-$Comp
-L power:+12V #PWR012
-U 1 1 61C07B21
-P 6800 2600
-F 0 "#PWR012" H 6800 2450 50  0001 C CNN
-F 1 "+12V" V 6815 2728 50  0000 L CNN
-F 2 "" H 6800 2600 50  0001 C CNN
-F 3 "" H 6800 2600 50  0001 C CNN
-	1    6800 2600
-	0    1    1    0
 $EndComp
 Wire Wire Line
@@
 L Mechanical:MountingHole_Pad H3
 U 1 1 61C0200E
-P 2050 5600
-F 0 "H3" V 2287 5603 50  0000 C CNN
-F 1 "MountingHole_Pad" V 2196 5603 50  0000 C CNN
-F 2 "MountingHole:MountingHole_3.2mm_M3_ISO7380_Pad" H 2050 5600 50  0001 C CNN
-F 3 "~" H 2050 5600 50  0001 C CNN
-	1    2050 5600
+P 2050 5550
+F 0 "H3" V 2287 5553 50  0000 C CNN
+F 1 "MountingHole_Pad" V 2196 5553 50  0000 C CNN
+F 2 "MountingHole:MountingHole_3.2mm_M3_ISO7380_Pad" H 2050 5550 50  0001 C CNN
+F 3 "~" H 2050 5550 50  0001 C CNN
+	1    2050 5550
 	0    -1   -1   0
 $EndComp
@@
 Wire Wire Line
 	9100 1300 9100 1400
-$Comp
-L power:+15V #PWR07
-U 1 1 61D52F32
-P 9850 2100
-F 0 "#PWR07" H 9850 1950 50  0001 C CNN
-F 1 "+15V" V 9865 2228 50  0000 L CNN
-F 2 "" H 9850 2100 50  0001 C CNN
-F 3 "" H 9850 2100 50  0001 C CNN
-	1    9850 2100
-	0    1    1    0
-$EndComp
 Wire Wire Line
 	9500 2100 9850 2100
@@
 	5600 1300 5100 1300
 Connection ~ 5600 1300
-$Comp
-L Connector:Conn_01x01_Female J3
-U 1 1 61D5085B
-P 7500 4050
-F 0 "J3" H 7392 3825 50  0000 C CNN
-F 1 "Conn_01x01_Female" H 7392 3916 50  0000 C CNN
-F 2 "_сustom:LUT_PinHeader_1x01_P2.54mm_Vertical" H 7500 4050 50  0001 C CNN
-F 3 "~" H 7500 4050 50  0001 C CNN
-	1    7500 4050
-	-1   0    0    1
-$EndComp
 Wire Wire Line
 	3700 1450 4200 1450
 Connection ~ 3700 1450
 Text GLabel 4200 1450 2    50   Input ~ 0
-Vin
-Text GLabel 7900 4050 2    50   Input ~ 0
-Vin
++19V
 Wire Wire Line
 	7700 4050 7900 4050
-$Comp
-L Connector:Conn_01x01_Female J4
-U 1 1 61D826F2
-P 7500 4400
-F 0 "J4" H 7392 4175 50  0000 C CNN
-F 1 "Conn_01x01_Female" H 7392 4266 50  0000 C CNN
-F 2 "_сustom:LUT_PinHeader_1x01_P2.54mm_Vertical" H 7500 4400 50  0001 C CNN
-F 3 "~" H 7500 4400 50  0001 C CNN
-	1    7500 4400
-	-1   0    0    1
-$EndComp
-Text GLabel 7900 4400 2    50   Input ~ 0
-Vin
 Wire Wire Line
 	7700 4400 7900 4400
@@
 Wire Wire Line
 	8550 4450 8700 4450
-$Comp
-L Connector:Conn_01x01_Female J1
-U 1 1 61DB7218
-P 8350 4050
-F 0 "J1" H 8242 3825 50  0000 C CNN
-F 1 "Conn_01x01_Female" H 8242 3916 50  0000 C CNN
-F 2 "_сustom:LUT_PinHeader_1x01_P2.54mm_Vertical" H 8350 4050 50  0001 C CNN
-F 3 "~" H 8350 4050 50  0001 C CNN
-	1    8350 4050
-	-1   0    0    1
-$EndComp
-$Comp
-L Connector:Conn_01x01_Female J2
-U 1 1 61DB9536
-P 8350 4450
-F 0 "J2" H 8242 4225 50  0000 C CNN
-F 1 "Conn_01x01_Female" H 8242 4316 50  0000 C CNN
-F 2 "_сustom:LUT_PinHeader_1x01_P2.54mm_Vertical" H 8350 4450 50  0001 C CNN
-F 3 "~" H 8350 4450 50  0001 C CNN
-	1    8350 4450
-	-1   0    0    1
-$EndComp
 Connection ~ 7100 1300
 $Comp
@@
 	1350 4000 1450 4000
 $Comp
-L power:+15V #PWR0102
-U 1 1 61D59D56
-P 1650 3200
-F 0 "#PWR0102" H 1650 3050 50  0001 C CNN
-F 1 "+15V" V 1665 3328 50  0000 L CNN
-F 2 "" H 1650 3200 50  0001 C CNN
-F 3 "" H 1650 3200 50  0001 C CNN
-	1    1650 3200
-	1    0    0    -1
-$EndComp
-$Comp
 L Device:R R10
 U 1 1 61D61660
@@
 Wire Wire Line
 	1000 4200 1000 4300
-Text Notes 950  1050 0    100  ~ 20
+Text Notes 850  1000 0    100  ~ 20
 Input Protection Board
 Wire Notes Line
 	750  750  750  2650
 Text GLabel 5100 1300 0    50   Input ~ 0
-Vin
++19V
 Text Notes 1950 3150 0    100  ~ 20
-+5v reference generator.
++5v reference generator
 Wire Notes Line
 	750  2800 4500 2800
@@
 Wire Notes Line
 	4500 2650 750  2650
-Text Notes 4950 1050 0    100  ~ 20
+Text Notes 4750 1000 0    100  ~ 20
 Power Supply Board
 Wire Notes Line
@@
 	1    5700 4450
 	1    0    0    -1
-$EndComp
-$Comp
-L power:+12V #PWR0105
-U 1 1 61FA7AE1
-P 5700 4150
-F 0 "#PWR0105" H 5700 4000 50  0001 C CNN
-F 1 "+12V" V 5715 4278 50  0000 L CNN
-F 2 "" H 5700 4150 50  0001 C CNN
-F 3 "" H 5700 4150 50  0001 C CNN
-	1    5700 4150
-	0    1    1    0
 $EndComp
 Wire Wire Line
@@
 	-1   0    0    -1
 $EndComp
-Text Notes 4850 3950 0    100  ~ 20
+Text Notes 4750 3900 0    100  ~ 20
 Interface
 Connection ~ 2150 3900
@@
 Wire Wire Line
 	3350 3900 3050 3900
-$Comp
-L power:+5V #PWR0106
-U 1 1 61D8CB4E
-P 3350 3900
-F 0 "#PWR0106" H 3350 3750 50  0001 C CNN
-F 1 "+5V" V 3365 4028 50  0000 L CNN
-F 2 "" H 3350 3900 50  0001 C CNN
-F 3 "" H 3350 3900 50  0001 C CNN
-	1    3350 3900
-	0    1    1    0
-$EndComp
 Wire Wire Line
 	3050 4300 3050 4400
@@
 	0    1    1    0
 $EndComp
-$Comp
-L power:+5V #PWR0109
-U 1 1 621620EB
-P 6750 4200
-F 0 "#PWR0109" H 6750 4050 50  0001 C CNN
-F 1 "+5V" V 6765 4328 50  0000 L CNN
-F 2 "" H 6750 4200 50  0001 C CNN
-F 3 "" H 6750 4200 50  0001 C CNN
-	1    6750 4200
-	0    1    1    0
-$EndComp
-$Comp
-L power:+15V #PWR0110
-U 1 1 6217A4CE
-P 6750 4400
-F 0 "#PWR0110" H 6750 4250 50  0001 C CNN
-F 1 "+15V" V 6765 4528 50  0000 L CNN
-F 2 "" H 6750 4400 50  0001 C CNN
-F 3 "" H 6750 4400 50  0001 C CNN
-	1    6750 4400
-	0    1    1    0
-$EndComp
 Wire Wire Line
 	6650 4400 6750 4400
@@
 L Mechanical:MountingHole_Pad H5
 U 1 1 61DBAF53
-P 2800 5600
-F 0 "H5" V 3037 5603 50  0000 C CNN
-F 1 "MountingHole_Pad" V 2946 5603 50  0000 C CNN
-F 2 "MountingHole:MountingHole_3.2mm_M3_ISO7380_Pad" H 2800 5600 50  0001 C CNN
-F 3 "~" H 2800 5600 50  0001 C CNN
-	1    2800 5600
+P 2800 5550
+F 0 "H5" V 3037 5553 50  0000 C CNN
+F 1 "MountingHole_Pad" V 2946 5553 50  0000 C CNN
+F 2 "MountingHole:MountingHole_3.2mm_M3_ISO7380_Pad" H 2800 5550 50  0001 C CNN
+F 3 "~" H 2800 5550 50  0001 C CNN
+	1    2800 5550
 	0    -1   -1   0
 $EndComp
@@
 	0    -1   -1   0
 $EndComp
+Text GLabel 6800 2600 2    50   Input ~ 0
++12V
+Text GLabel 9850 2100 2    50   Input ~ 0
++15V
+Text GLabel 5700 4150 2    50   Input ~ 0
++12V
+Text GLabel 6750 4400 2    50   Input ~ 0
++15V
+Text GLabel 7900 4050 2    50   Input ~ 0
++19V
+Text GLabel 7900 4400 2    50   Input ~ 0
++19V
+$Comp
+L Connector_Generic:Conn_01x01 J1
+U 1 1 61E07297
+P 7500 4050
+F 0 "J1" H 7418 3825 50  0000 C CNN
+F 1 "Conn_01x01" H 7418 3916 50  0000 C CNN
+F 2 "_сustom:LUT_PinHeader_1x01_P2.54mm_Vertical" H 7500 4050 50  0001 C CNN
+F 3 "~" H 7500 4050 50  0001 C CNN
+	1    7500 4050
+	-1   0    0    1
+$EndComp
+$Comp
+L Connector_Generic:Conn_01x01 J3
+U 1 1 61E07E7C
+P 7500 4400
+F 0 "J3" H 7418 4175 50  0000 C CNN
+F 1 "Conn_01x01" H 7418 4266 50  0000 C CNN
+F 2 "_сustom:LUT_PinHeader_1x01_P2.54mm_Vertical" H 7500 4400 50  0001 C CNN
+F 3 "~" H 7500 4400 50  0001 C CNN
+	1    7500 4400
+	-1   0    0    1
+$EndComp
+$Comp
+L Connector_Generic:Conn_01x01 J2
+U 1 1 61E0B232
+P 8350 4050
+F 0 "J2" H 8268 3825 50  0000 C CNN
+F 1 "Conn_01x01" H 8268 3916 50  0000 C CNN
+F 2 "_сustom:LUT_PinHeader_1x01_P2.54mm_Vertical" H 8350 4050 50  0001 C CNN
+F 3 "~" H 8350 4050 50  0001 C CNN
+	1    8350 4050
+	-1   0    0    1
+$EndComp
+$Comp
+L Connector_Generic:Conn_01x01 J4
+U 1 1 61E0E515
+P 8350 4450
+F 0 "J4" H 8268 4225 50  0000 C CNN
+F 1 "Conn_01x01" H 8268 4316 50  0000 C CNN
+F 2 "_сustom:LUT_PinHeader_1x01_P2.54mm_Vertical" H 8350 4450 50  0001 C CNN
+F 3 "~" H 8350 4450 50  0001 C CNN
+	1    8350 4450
+	-1   0    0    1
+$EndComp
+Text GLabel 1650 3200 1    50   Input ~ 0
++15V
+Text GLabel 3350 3900 2    50   Input ~ 0
++5V
+Text GLabel 6750 4200 2    50   Input ~ 0
++5V
 $EndSCHEMATC
